Commit message: renaming package

File: gezengec_description/urdf/bumperbot.urdf.xacro (robot description, xacro)
@@ -1,5 +1,5 @@
 <?xml version="1.0"?>
 <robot name="bumperbot" xmlns:xacro="http://ros.org/wiki/xacro">
-  <xacro:include filename="$(find bumperbot_description)/urdf/bumperbot_gazebo.xacro"/>
+  <xacro:include filename="$(find gezengec_description)/urdf/bumperbot_gazebo.xacro"/>
   <link name="base_footprint"/>
   <link name="base_link">
@@ -14,5 +14,5 @@
       <origin xyz="0 0 0" rpy="0 0 0" />
       <geometry>
-        <mesh filename="package://bumperbot_description/meshes/base_link.STL" />
+        <mesh filename="package://gezengec_description/meshes/base_link.STL" />
       </geometry>
     </visual>
@@ -20,5 +20,5 @@
       <origin xyz="0 0 0" rpy="0 0 0" />
       <geometry>
-        <mesh filename="package://bumperbot_description/meshes/base_link.STL" />
+        <mesh filename="package://gezengec_description/meshes/base_link.STL" />
       </geometry>
     </collision>
@@ -40,5 +40,5 @@
       <origin xyz="0 0 0" rpy="1.57 0 0" />
       <geometry>
-        <mesh filename="package://bumperbot_description/meshes/wheel_right_link.STL" />
+        <mesh filename="package://gezengec_description/meshes/wheel_right_link.STL" />
       </geometry>
     </visual>
@@ -68,5 +68,5 @@
       <origin xyz="0 0 0" rpy="-1.57 0 0" />
       <geometry>
-        <mesh filename="package://bumperbot_description/meshes/wheel_left_link.STL" />
+        <mesh filename="package://gezengec_description/meshes/wheel_left_link.STL" />
       </geometry>
     </visual>
@@ -95,5 +95,5 @@
       <origin xyz="0 0 0" rpy="0 0 0" />
       <geometry>
-        <mesh filename="package://bumperbot_description/meshes/caster_front_link.STL" />
+        <mesh filename="package://gezengec_description/meshes/caster_front_link.STL" />
       </geometry>
     </visual>
@@ -122,5 +122,5 @@
       <origin xyz="0 0 0" rpy="0 0 0" />
       <geometry>
-        <mesh filename="package://bumperbot_description/meshes/caster_rear_link.STL" />
+        <mesh filename="package://gezengec_description/meshes/caster_rear_link.STL" />
       </geometry>
     </visual>

Commit message: adding plugins

File: gezengec_description/urdf/bumperbot.urdf.xacro (robot description, xacro)
@@ -138,3 +138,30 @@
     <axis xyz="0 0 0" />
   </joint>
+  <link name="imu_link">
+    <inertial>
+      <origin xyz="-0.00552433659106688 0.000168210391520346 0.000514000497342681" rpy="0 0 0" />
+      <mass value="0.000528415362211671" />
+      <inertia ixx="1.46176048428261E-08" ixy="1.40015117949421E-10" ixz="-1.99633872937403E-12"
+                iyy="8.59662482954888E-09" iyz="7.52375112767959E-12"
+                izz="2.30279421279312E-08" />
+    </interial>
+    <visual>
+      <origin xyz="0 0 0" rpy= "0 0 0"/>
+      <geometry>
+        <mesh filename="package://gezengec_description/meshes/imu_link.STL">
+      </geometry>
+    </visual>
+    <collision>
+      <origin xyz="0 0 0" rpy= "0 0 0"/>
+      <geometry>
+        <mesh filename="package://gezengec_description/meshes/imu_link.STL">
+      </geometry>
+    </collision>
+  </link>
+  <joint name="imu_joint" type="fixed">
+        <origin xyz="0 0 0.07" rpy="3.14 0 0"/>
+        <parent link="base_link"/>
+        <child link="imu_link"/>
+        <axis xyz="0 0 0"/>
+  </joint>
 </robot>

File: gezengec_description/urdf/bumperbot_gazebo.xacro (robot description, xacro)
@@ -35,3 +35,18 @@
     <maxVel>1.0</maxVel>
   </gazebo>
+  <gazebo>
+    <plugin name="gazebo_ros_control" filename="libgazebo_ros_control.so">
+      <robotSimType>gazebo_ros_control/DefaultRobotHWSim</robotSimType>
+      <legacyModeNS>true</legacyModeNS>
+  </gazebo>
+  <gazebo>
+    <plugin name="imu_plugin" filename="libgazebo_ros_imu.so">
+      <alwaysOn>true</alwaysOn>
+      <bodyName>imu_link</bodyName>
+      <frameName>imu_link</frameName>
+      <topic_name>imu</topic_name>
+      <serviceName>imu_service</serviceName>
+      <gaussianNoise>0.001</gaussianNoise>
+      <updateRate>1000</updateRate>
+  </gazebo>
 </robot>

Commit message: fixing errors

File: gezengec_description/urdf/bumperbot.urdf.xacro (robot description, xacro)
@@ -144,10 +144,10 @@
       <inertia ixx="1.46176048428261E-08" ixy="1.40015117949421E-10" ixz="-1.99633872937403E-12"
                 iyy="8.59662482954888E-09" iyz="7.52375112767959E-12"
-                izz="2.30279421279312E-08" />
-    </interial>
+                izz="2.30279421279312E-08"/>
+    </inertial>
     <visual>
       <origin xyz="0 0 0" rpy= "0 0 0"/>
       <geometry>
-        <mesh filename="package://gezengec_description/meshes/imu_link.STL">
+        <mesh filename="package://gezengec_description/meshes/imu_link.STL"/>
       </geometry>
     </visual>
@@ -155,5 +155,5 @@
       <origin xyz="0 0 0" rpy= "0 0 0"/>
       <geometry>
-        <mesh filename="package://gezengec_description/meshes/imu_link.STL">
+        <mesh filename="package://gezengec_description/meshes/imu_link.STL"/>
       </geometry>
     </collision>

File: gezengec_description/urdf/bumperbot_gazebo.xacro (robot description, xacro)
@@ -39,4 +39,5 @@
       <robotSimType>gazebo_ros_control/DefaultRobotHWSim</robotSimType>
       <legacyModeNS>true</legacyModeNS>
+    </plugin>
   </gazebo>
   <gazebo>
@@ -49,4 +50,5 @@
       <gaussianNoise>0.001</gaussianNoise>
       <updateRate>1000</updateRate>
+    </plugin>
   </gazebo>
 </robot>

Commit message: updating xacro files

File: gezengec_description/urdf/bumperbot.urdf.xacro (robot description, xacro)
@@ -1,5 +1,5 @@
 <?xml version="1.0"?>
 <robot name="bumperbot" xmlns:xacro="http://ros.org/wiki/xacro">
-  <xacro:include filename="$(find gezengec_description)/urdf/bumperbot_gazebo.xacro"/>
+  <xacro:include filename="$(find bumperbot_description)/urdf/bumperbot_gazebo.xacro"/>
   <link name="base_footprint"/>
   <link name="base_link">
@@ -14,5 +14,5 @@
       <origin xyz="0 0 0" rpy="0 0 0" />
       <geometry>
-        <mesh filename="package://gezengec_description/meshes/base_link.STL" />
+        <mesh filename="package://bumperbot_description/meshes/base_link.STL" />
       </geometry>
     </visual>
@@ -20,5 +20,5 @@
       <origin xyz="0 0 0" rpy="0 0 0" />
       <geometry>
-        <mesh filename="package://gezengec_description/meshes/base_link.STL" />
+        <mesh filename="package://bumperbot_description/meshes/base_link.STL" />
       </geometry>
     </collision>
@@ -40,5 +40,5 @@
       <origin xyz="0 0 0" rpy="1.57 0 0" />
       <geometry>
-        <mesh filename="package://gezengec_description/meshes/wheel_right_link.STL" />
+        <mesh filename="package://bumperbot_description/meshes/wheel_right_link.STL" />
       </geometry>
     </visual>
@@ -68,5 +68,5 @@
       <origin xyz="0 0 0" rpy="-1.57 0 0" />
       <geometry>
-        <mesh filename="package://gezengec_description/meshes/wheel_left_link.STL" />
+        <mesh filename="package://bumperbot_description/meshes/wheel_left_link.STL" />
       </geometry>
     </visual>
@@ -95,5 +95,5 @@
       <origin xyz="0 0 0" rpy="0 0 0" />
       <geometry>
-        <mesh filename="package://gezengec_description/meshes/caster_front_link.STL" />
+        <mesh filename="package://bumperbot_description/meshes/caster_front_link.STL" />
       </geometry>
     </visual>
@@ -122,5 +122,5 @@
       <origin xyz="0 0 0" rpy="0 0 0" />
       <geometry>
-        <mesh filename="package://gezengec_description/meshes/caster_rear_link.STL" />
+        <mesh filename="package://bumperbot_description/meshes/caster_rear_link.STL" />
       </geometry>
     </visual>
@@ -143,25 +143,25 @@
       <mass value="0.000528415362211671" />
       <inertia ixx="1.46176048428261E-08" ixy="1.40015117949421E-10" ixz="-1.99633872937403E-12"
-                iyy="8.59662482954888E-09" iyz="7.52375112767959E-12"
-                izz="2.30279421279312E-08"/>
+               iyy="8.59662482954888E-09" iyz="7.52375112767959E-12"
+               izz="2.30279421279312E-08" />
     </inertial>
     <visual>
-      <origin xyz="0 0 0" rpy= "0 0 0"/>
+      <origin xyz="0 0 0" rpy="0 0 0" />
       <geometry>
-        <mesh filename="package://gezengec_description/meshes/imu_link.STL"/>
+        <mesh filename="package://bumperbot_description/meshes/imu_link.STL" />
       </geometry>
     </visual>
     <collision>
-      <origin xyz="0 0 0" rpy= "0 0 0"/>
+      <origin xyz="0 0 0" rpy="0 0 0" />
       <geometry>
-        <mesh filename="package://gezengec_description/meshes/imu_link.STL"/>
+        <mesh filename="package://bumperbot_description/meshes/imu_link.STL" />
       </geometry>
     </collision>
   </link>
   <joint name="imu_joint" type="fixed">
-        <origin xyz="0 0 0.07" rpy="3.14 0 0"/>
-        <parent link="base_link"/>
-        <child link="imu_link"/>
-        <axis xyz="0 0 0"/>
+    <origin xyz="0 0 0.0698986241758014" rpy="3.14159265358979 0 0" />
+    <parent link="base_link" />
+    <child link="imu_link" />
+    <axis xyz="0 0 0" />
   </joint>
 </robot>

File: gezengec_description/urdf/bumperbot_gazebo.xacro (robot description, xacro)
@@ -55,4 +55,5 @@
     <maxVel>1.0</maxVel>
   </gazebo>
+  <!-- ROS Control -->
   <gazebo>
     <plugin name="gazebo_ros_control" filename="libgazebo_ros_control.so">
@@ -61,4 +62,5 @@
     </plugin>
   </gazebo>
+  <!-- IMU -->
   <gazebo>
     <plugin name="imu_plugin" filename="libgazebo_ros_imu.so">

Commit message: updating xacro files

File: gezengec_description/urdf/bumperbot.urdf.xacro (robot description, xacro)
@@ -1,5 +1,5 @@
 <?xml version="1.0"?>
 <robot name="bumperbot" xmlns:xacro="http://ros.org/wiki/xacro">
-  <xacro:include filename="$(find bumperbot_description)/urdf/bumperbot_gazebo.xacro"/>
+  <xacro:include filename="$(find gezengec_description)/urdf/bumperbot_gazebo.xacro"/>
   <link name="base_footprint"/>
   <link name="base_link">
@@ -14,5 +14,5 @@
       <origin xyz="0 0 0" rpy="0 0 0" />
       <geometry>
-        <mesh filename="package://bumperbot_description/meshes/base_link.STL" />
+        <mesh filename="package://gezengec_description/meshes/base_link.STL" />
       </geometry>
     </visual>
@@ -20,5 +20,5 @@
       <origin xyz="0 0 0" rpy="0 0 0" />
       <geometry>
-        <mesh filename="package://bumperbot_description/meshes/base_link.STL" />
+        <mesh filename="package://gezengec_description/meshes/base_link.STL" />
       </geometry>
     </collision>
@@ -40,5 +40,5 @@
       <origin xyz="0 0 0" rpy="1.57 0 0" />
       <geometry>
-        <mesh filename="package://bumperbot_description/meshes/wheel_right_link.STL" />
+        <mesh filename="package://gezengec_description/meshes/wheel_right_link.STL" />
       </geometry>
     </visual>
@@ -68,5 +68,5 @@
       <origin xyz="0 0 0" rpy="-1.57 0 0" />
       <geometry>
-        <mesh filename="package://bumperbot_description/meshes/wheel_left_link.STL" />
+        <mesh filename="package://gezengec_description/meshes/wheel_left_link.STL" />
       </geometry>
     </visual>
@@ -95,5 +95,5 @@
       <origin xyz="0 0 0" rpy="0 0 0" />
       <geometry>
-        <mesh filename="package://bumperbot_description/meshes/caster_front_link.STL" />
+        <mesh filename="package://gezengec_description/meshes/caster_front_link.STL" />
       </geometry>
     </visual>
@@ -122,5 +122,5 @@
       <origin xyz="0 0 0" rpy="0 0 0" />
       <geometry>
-        <mesh filename="package://bumperbot_description/meshes/caster_rear_link.STL" />
+        <mesh filename="package://gezengec_description/meshes/caster_rear_link.STL" />
       </geometry>
     </visual>
@@ -149,5 +149,5 @@
       <origin xyz="0 0 0" rpy="0 0 0" />
       <geometry>
-        <mesh filename="package://bumperbot_description/meshes/imu_link.STL" />
+        <mesh filename="package://gezengec_description/meshes/imu_link.STL" />
       </geometry>
     </visual>
@@ -155,5 +155,5 @@
       <origin xyz="0 0 0" rpy="0 0 0" />
       <geometry>
-        <mesh filename="package://bumperbot_description/meshes/imu_link.STL" />
+        <mesh filename="package://gezengec_description/meshes/imu_link.STL" />
       </geometry>
     </collision>
