Commit message: fixing errors

File: gezengec_description/urdf/gezengec.urdf.xacro (robot description, xacro)
@@ -1,5 +1,5 @@
 <?xml version="1.0"?>
-<robot name="bumperbot" xmlns:xacro="http://ros.org/wiki/xacro">
-  <xacro:include filename="$(find gezengec_description)/urdf/bumperbot_gazebo.xacro"/>
+<robot name="gezengec" xmlns:xacro="http://ros.org/wiki/xacro">
+  <xacro:include filename="$(find gezengec_description)/urdf/gezengec_gazebo.xacro"/>
   <link name="base_footprint"/>
   <link name="base_link">
@@ -24,4 +24,7 @@
     </collision>
   </link>
+  <gazebo reference="base_link">
+    <material>Gazebo/Yellow</material>
+  </gazebo>
   <joint name="base_joint" type="fixed">
     <parent link="base_footprint"/>
@@ -50,4 +53,7 @@
     </collision>
   </link>
+  <gazebo reference="wheel_right_link">
+    <material>Gazebo/Gray</material>
+  </gazebo>
   <joint name="wheel_right_joint" type="continuous">
     <origin xyz="0 -0.0701101849418637 0" rpy="0 0 0" />
@@ -78,4 +84,7 @@
     </collision>
   </link>
+  <gazebo reference="wheel_left_link">
+    <material>Gazebo/Gray</material>
+  </gazebo>
   <joint name="wheel_left_joint" type="continuous">
     <origin xyz="0 0.0701101849418642 0" rpy="0 0 0" />

File: gezengec_description/urdf/gezengec_gazebo.xacro (robot description, xacro)
@@ -1,4 +1,4 @@
 <?xml version="1.0"?>
-<robot name="bumperbot" xmlns:xacro="http://ros.org/wiki/xacro">
+<robot name="gezengec" xmlns:xacro="http://ros.org/wiki/xacro">
   <transmission name="wheel_right_transmission">
     <type>transmission_interface/SimpleTransmission</type>
